Commit message: 12

File: urdf/12-gripper.urdf.xacro (robot description, xacro)
@@ -1,4 +1,4 @@
 <?xml version="1.0"?>
-<robot name="r2d2" xmlns:xacro="http://ros.org/wiki/xacro">
+<robot name="gripper_controller" xmlns:xacro="http://ros.org/wiki/xacro">
   <xacro:property name="width" value="0.2" />
   <xacro:property name="leglen" value="0.6" />
@@ -7,5 +7,4 @@
   <xacro:property name="baselen" value="0.4" />
   <xacro:property name="wheeldiam" value="0.07" />
-  <xacro:property name="pi" value="3.1415" />
   <material name="blue">
     <color rgba="0 0 0.8 1"/>
@@ -20,5 +19,5 @@
     <inertial>
       <mass value="${mass}" />
-      <inertia ixx="1.0" ixy="0.0" ixz="0.0" iyy="1.0" iyz="0.0" izz="1.0" />
+      <inertia ixx="1e-3" ixy="0.0" ixz="0.0" iyy="1e-3" iyz="0.0" izz="1e-3" />
     </inertial>
   </xacro:macro>
@@ -130,13 +129,4 @@
     <xacro:default_inertial mass="0.05"/>
   </link>
-  <transmission name="gripper_extension_trans" type="SimpleTransmission">
-    <type>transmission_interface/SimpleTransmission</type>
-    <actuator name="gripper_extension_motor">
-      <mechanicalReduction>1</mechanicalReduction>
-    </actuator>
-    <joint name="gripper_extension">
-      <hardwareInterface>PositionJointInterface</hardwareInterface>
-    </joint>
-  </transmission>
   <xacro:macro name="gripper" params="prefix reflect">
     <joint name="${prefix}_gripper_joint" type="revolute">
@@ -164,13 +154,4 @@
       <xacro:default_inertial mass="0.05"/>
     </link>
-    <transmission name="${prefix}_gripper_trans" type="SimpleTransmission">
-      <type>transmission_interface/SimpleTransmission</type>
-      <actuator name="${prefix}_gripper_motor">
-        <mechanicalReduction>1</mechanicalReduction>
-      </actuator>
-      <joint name="${prefix}_gripper_joint">
-        <hardwareInterface>PositionJointInterface</hardwareInterface>
-      </joint>
-    </transmission>
     <joint name="${prefix}_tip_joint" type="fixed">
       <parent link="${prefix}_gripper"/>
@@ -217,15 +198,4 @@
     <dynamics damping="0.0" friction="0.0"/>
   </joint>
-  <!-- This block connects the head_swivel joint to an actuator (motor), which informs both
-  simulation and visualization of the robot -->
-  <transmission name="head_swivel_trans">
-    <type>transmission_interface/SimpleTransmission</type>
-    <actuator name="$head_swivel_motor">
-      <mechanicalReduction>1</mechanicalReduction>
-    </actuator>
-    <joint name="head_swivel">
-      <hardwareInterface>PositionJointInterface</hardwareInterface>
-    </joint>
-  </transmission>
   <link name="box">
     <visual>
@@ -248,8 +218,36 @@
     <origin xyz="${.707*width+0.04} 0 ${.707*width}"/>
   </joint>
-  <!-- Gazebo plugin for ROS Control -->
+  <ros2_control name="GazeboSystem" type="system">
+    <hardware>
+      <plugin>gazebo_ros2_control/GazeboSystem</plugin>
+    </hardware>
+    <joint name="head_swivel">
+      <command_interface name="position" />
+      <command_interface name="velocity" />
+      <state_interface name="position"/>
+      <state_interface name="velocity"/>
+    </joint>
+    <joint name="gripper_extension">
+      <command_interface name="position" />
+      <command_interface name="velocity" />
+      <state_interface name="position"/>
+      <state_interface name="velocity"/>
+    </joint>
+    <joint name="left_gripper_joint">
+      <command_interface name="position" />
+      <command_interface name="velocity" />
+      <state_interface name="position"/>
+      <state_interface name="velocity"/>
+    </joint>
+    <joint name="right_gripper_joint">
+      <command_interface name="position" />
+      <command_interface name="velocity" />
+      <state_interface name="position"/>
+      <state_interface name="velocity"/>
+    </joint>
+  </ros2_control>
   <gazebo>
-    <plugin name="gazebo_ros_control" filename="libgazebo_ros_control.so">
-      <robotNamespace>/</robotNamespace>
+    <plugin filename="libgazebo_ros2_control.so" name="gazebo_ros2_control">
+      <parameters>$(find urdf_sim_tutorial)/config/gripper.yaml</parameters>
     </plugin>
   </gazebo>
