Commit message: added gazebo material tag in xacro

File: urdf/13-diffdrive.urdf.xacro (robot description, xacro)
@@ -36,4 +36,7 @@
     <xacro:default_inertial mass="10"/>
   </link>
+  <gazebo reference="base_link">
+    <material>Gazebo/Blue</material>
+  </gazebo>
   <xacro:macro name="wheel" params="prefix suffix reflect">
     <link name="${prefix}_${suffix}_wheel">
@@ -121,4 +124,10 @@
       <origin xyz="0 0 ${-leglen}" />
     </joint>
+    <gazebo reference="${prefix}_leg">
+      <material>Gazebo/White</material>
+    </gazebo>
+    <gazebo reference="${prefix}_base">
+      <material>Gazebo/White</material>
+    </gazebo>
     <xacro:wheel prefix="${prefix}" suffix="front" reflect="1"/>
     <xacro:wheel prefix="${prefix}" suffix="back" reflect="-1"/>
@@ -149,4 +158,7 @@
     <xacro:default_inertial mass="0.05"/>
   </link>
+  <gazebo reference="gripper_pole">
+    <material>Gazebo/Red</material>
+  </gazebo>
   <transmission name="gripper_extension_trans">
     <type>transmission_interface/SimpleTransmission</type>
@@ -236,4 +248,7 @@
     <dynamics damping="0.0" friction="0.0"/>
   </joint>
+  <gazebo reference="head">
+    <material>Gazebo/White</material>
+  </gazebo>
   <!-- This block connects the head_swivel joint to an actuator (motor), which informs both
   simulation and visualization of the robot -->
@@ -267,4 +282,7 @@
     <origin xyz="${.707*width+0.04} 0 ${.707*width}"/>
   </joint>
+  <gazebo reference="box">
+    <material>Gazebo/Blue</material>
+  </gazebo>
   <!-- Gazebo plugin for ROS Control -->
   <gazebo>

Commit message: 13 basic

File: urdf/13-diffdrive.urdf.xacro (robot description, xacro)
@@ -1,4 +1,4 @@
 <?xml version="1.0"?>
-<robot name="roscontrol" xmlns:xacro="http://ros.org/wiki/xacro">
+<robot name="diff_drive" xmlns:xacro="http://ros.org/wiki/xacro">
   <xacro:property name="width" value="0.2" />
   <xacro:property name="leglen" value="0.6" />
@@ -7,5 +7,4 @@
   <xacro:property name="baselen" value="0.4" />
   <xacro:property name="wheeldiam" value="0.07" />
-  <xacro:property name="pi" value="3.1415" />
   <material name="blue">
     <color rgba="0 0 0.8 1"/>
@@ -20,5 +19,5 @@
     <inertial>
       <mass value="${mass}" />
-      <inertia ixx="1.0" ixy="0.0" ixz="0.0" iyy="1.0" iyz="0.0" izz="1.0" />
+      <inertia ixx="1e-3" ixy="0.0" ixz="0.0" iyy="1e-3" iyz="0.0" izz="1e-3" />
     </inertial>
   </xacro:macro>
@@ -69,15 +68,4 @@
       <material>Gazebo/Grey</material>
     </gazebo>
-    <!-- This block connects the wheel joint to an actuator (motor), which informs both
-    simulation and visualization of the robot -->
-    <transmission name="${prefix}_${suffix}_wheel_trans">
-      <type>transmission_interface/SimpleTransmission</type>
-      <actuator name="${prefix}_${suffix}_wheel_motor">
-        <mechanicalReduction>1</mechanicalReduction>
-      </actuator>
-      <joint name="${prefix}_${suffix}_wheel_joint">
-        <hardwareInterface>VelocityJointInterface</hardwareInterface>
-      </joint>
-    </transmission>
   </xacro:macro>
   <xacro:macro name="leg" params="prefix reflect">
@@ -150,15 +138,7 @@
     <xacro:default_inertial mass="0.05"/>
   </link>
-  <transmission name="gripper_extension_trans">
-    <type>transmission_interface/SimpleTransmission</type>
-    <actuator name="gripper_extension_motor">
-      <mechanicalReduction>1</mechanicalReduction>
-    </actuator>
-    <joint name="gripper_extension">
-      <hardwareInterface>PositionJointInterface</hardwareInterface>
-    </joint>
-  </transmission>
-  <xacro:macro name="gripper" params="prefix reflect">
+  <xacro:macro name="gripper" params="prefix reflect *extra_tag">
     <joint name="${prefix}_gripper_joint" type="revolute">
+      <xacro:insert_block name="extra_tag" />
       <axis xyz="0 0 ${reflect}"/>
       <limit effort="1000.0" lower="0.0" upper="0.548" velocity="0.5"/>
@@ -184,13 +164,4 @@
       <xacro:default_inertial mass="0.05"/>
     </link>
-    <transmission name="${prefix}_gripper_trans">
-      <type>transmission_interface/SimpleTransmission</type>
-      <actuator name="${prefix}_gripper_motor">
-        <mechanicalReduction>1</mechanicalReduction>
-      </actuator>
-      <joint name="${prefix}_gripper_joint">
-        <hardwareInterface>PositionJointInterface</hardwareInterface>
-      </joint>
-    </transmission>
     <joint name="${prefix}_tip_joint" type="fixed">
       <parent link="${prefix}_gripper"/>
@@ -213,6 +184,10 @@
     </link>
   </xacro:macro>
-  <xacro:gripper prefix="left" reflect="1" />
-  <xacro:gripper prefix="right" reflect="-1" />
+  <xacro:gripper prefix="left" reflect="1">
+    <dynamics damping="0.0" friction="0.0"/>
+  </xacro:gripper>
+  <xacro:gripper prefix="right" reflect="-1">
+     <mimic joint="left_gripper_joint"/>
+  </xacro:gripper>
   <link name="head">
     <visual>
@@ -237,15 +212,4 @@
     <dynamics damping="0.0" friction="0.0"/>
   </joint>
-  <!-- This block connects the head_swivel joint to an actuator (motor), which informs both
-  simulation and visualization of the robot -->
-  <transmission name="head_swivel_trans">
-    <type>transmission_interface/SimpleTransmission</type>
-    <actuator name="$head_swivel_motor">
-      <mechanicalReduction>1</mechanicalReduction>
-    </actuator>
-    <joint name="head_swivel">
-      <hardwareInterface>PositionJointInterface</hardwareInterface>
-    </joint>
-  </transmission>
   <link name="box">
     <visual>
@@ -268,8 +232,62 @@
     <origin xyz="${.707*width+0.04} 0 ${.707*width}"/>
   </joint>
-  <!-- Gazebo plugin for ROS Control -->
+  <ros2_control name="GazeboSystem" type="system">
+    <hardware>
+      <plugin>gazebo_ros2_control/GazeboSystem</plugin>
+    </hardware>
+    <joint name="head_swivel">
+      <command_interface name="position" />
+      <command_interface name="velocity" />
+      <state_interface name="position"/>
+      <state_interface name="velocity"/>
+    </joint>
+    <joint name="gripper_extension">
+      <command_interface name="position" />
+      <command_interface name="velocity" />
+      <state_interface name="position"/>
+      <state_interface name="velocity"/>
+    </joint>
+    <joint name="left_gripper_joint">
+      <command_interface name="position" />
+      <command_interface name="velocity" />
+      <state_interface name="position"/>
+      <state_interface name="velocity"/>
+    </joint>
+    <joint name="right_gripper_joint">
+      <command_interface name="position" />
+      <command_interface name="velocity" />
+      <state_interface name="position"/>
+      <state_interface name="velocity"/>
+      <param name="mimic">left_gripper_joint</param>
+      <param name="multiplier">1</param>
+    </joint>
+    <joint name="left_front_wheel_joint">
+      <command_interface name="position" />
+      <command_interface name="velocity" />
+      <state_interface name="position"/>
+      <state_interface name="velocity"/>
+    </joint>
+    <joint name="left_back_wheel_joint">
+      <command_interface name="position" />
+      <command_interface name="velocity" />
+      <state_interface name="position"/>
+      <state_interface name="velocity"/>
+    </joint>
+    <joint name="right_front_wheel_joint">
+      <command_interface name="position" />
+      <command_interface name="velocity" />
+      <state_interface name="position"/>
+      <state_interface name="velocity"/>
+    </joint>
+    <joint name="right_back_wheel_joint">
+      <command_interface name="position" />
+      <command_interface name="velocity" />
+      <state_interface name="position"/>
+      <state_interface name="velocity"/>
+    </joint>
+  </ros2_control>
   <gazebo>
-    <plugin name="gazebo_ros_control" filename="libgazebo_ros_control.so">
-      <robotNamespace>/</robotNamespace>
+    <plugin filename="libgazebo_ros2_control.so" name="gazebo_ros2_control">
+      <parameters>$(find urdf_sim_tutorial)/config/diffdrive.yaml</parameters>
     </plugin>
   </gazebo>

Commit message: Partial Diff Drive

File: urdf/13-diffdrive.urdf.xacro (robot description, xacro)
@@ -59,13 +59,4 @@
       <origin xyz="${baselen*reflect/3} 0 -${wheeldiam/2+.05}" rpy="0 0 0"/>
     </joint>
-    <!-- This block provides the simulator (Gazebo) with information on a few additional
-    physical properties. See http://gazebosim.org/tutorials/?tut=ros_urdf for more-->
-    <gazebo reference="${prefix}_${suffix}_wheel">
-      <mu1 value="200.0"/>
-      <mu2 value="100.0"/>
-      <kp value="10000000.0" />
-      <kd value="1.0" />
-      <material>Gazebo/Grey</material>
-    </gazebo>
   </xacro:macro>
   <xacro:macro name="leg" params="prefix reflect">
