Commit message: Remove Pi constant

File: urdf/09-publishjoints.urdf.xacro (robot description, xacro)
@@ -7,5 +7,4 @@
   <xacro:property name="baselen" value="0.4" />
   <xacro:property name="wheeldiam" value="0.07" />
-  <xacro:property name="pi" value="3.1415" />
   <material name="blue">
     <color rgba="0 0 0.8 1"/>

File: urdf/10-firsttransmission.urdf.xacro (robot description, xacro)
@@ -7,5 +7,4 @@
   <xacro:property name="baselen" value="0.4" />
   <xacro:property name="wheeldiam" value="0.07" />
-  <xacro:property name="pi" value="3.1415" />
   <material name="blue">
     <color rgba="0 0 0.8 1"/>

File: urdf/11-limittransmission.urdf.xacro (robot description, xacro)
@@ -7,5 +7,4 @@
   <xacro:property name="baselen" value="0.4" />
   <xacro:property name="wheeldiam" value="0.07" />
-  <xacro:property name="pi" value="3.1415" />
   <material name="blue">
     <color rgba="0 0 0.8 1"/>

File: urdf/12-gripper.urdf.xacro (robot description, xacro)
@@ -7,5 +7,4 @@
   <xacro:property name="baselen" value="0.4" />
   <xacro:property name="wheeldiam" value="0.07" />
-  <xacro:property name="pi" value="3.1415" />
   <material name="blue">
     <color rgba="0 0 0.8 1"/>

File: urdf/13-diffdrive.urdf.xacro (robot description, xacro)
@@ -7,5 +7,4 @@
   <xacro:property name="baselen" value="0.4" />
   <xacro:property name="wheeldiam" value="0.07" />
-  <xacro:property name="pi" value="3.1415" />
   <material name="blue">
     <color rgba="0 0 0.8 1"/>

Commit message: Convert Tutorial to ROS 2 (#13)
* Initial conversion

* 9 and 10

* 10 and 11

* 12

* Mimic Tag

* 13 basic

* Update rviz

* Partial Diff Drive

* Diff Drive

* Apply suggestions from code review

Co-authored-by: Alejandro Hernández Cordero <ahcorde@gmail.com>

* Add license to launch files

* Use environment variable for distro

* PathJoinSubstitution

* Precommit Configuration

* Change ``` to indent

* Add setup.cfg

---------

Co-authored-by: Alejandro Hernández Cordero <ahcorde@gmail.com>

File: urdf/09-publishjoints.urdf.xacro (robot description, xacro)
@@ -7,5 +7,4 @@
   <xacro:property name="baselen" value="0.4" />
   <xacro:property name="wheeldiam" value="0.07" />
-  <xacro:property name="pi" value="3.1415" />
   <material name="blue">
     <color rgba="0 0 0.8 1"/>
@@ -20,5 +19,5 @@
     <inertial>
       <mass value="${mass}" />
-      <inertia ixx="1.0" ixy="0.0" ixz="0.0" iyy="1.0" iyz="0.0" izz="1.0" />
+      <inertia ixx="1e-3" ixy="0.0" ixz="0.0" iyy="1e-3" iyz="0.0" izz="1e-3" />
     </inertial>
   </xacro:macro>
@@ -213,8 +212,13 @@
     <origin xyz="${.707*width+0.04} 0 ${.707*width}"/>
   </joint>
-  <!-- Gazebo plugin for ROS Control -->
+  <ros2_control name="GazeboSystem" type="system">
+    <hardware>
+      <plugin>gazebo_ros2_control/GazeboSystem</plugin>
+    </hardware>
+    <joint name="head_swivel" />
+  </ros2_control>
   <gazebo>
-    <plugin name="gazebo_ros_control" filename="libgazebo_ros_control.so">
-      <robotNamespace>/</robotNamespace>
+    <plugin filename="libgazebo_ros2_control.so" name="gazebo_ros2_control">
+      <parameters>$(find urdf_sim_tutorial)/config/joints.yaml</parameters>
     </plugin>
   </gazebo>

File: urdf/09a-minimal.urdf.xacro (robot description, xacro)
@@ -1,4 +1,4 @@
 <?xml version="1.0"?>
-<robot name="first_transmission_with_limits" xmlns:xacro="http://ros.org/wiki/xacro">
+<robot name="gazebo1" xmlns:xacro="http://ros.org/wiki/xacro">
   <xacro:property name="width" value="0.2" />
   <xacro:property name="leglen" value="0.6" />
@@ -191,5 +191,4 @@
     <axis xyz="0 0 1"/>
     <origin xyz="0 0 ${bodylen/2}"/>
-    <limit effort="30" velocity="1.0"/>
   </joint>
   <link name="box">
@@ -217,14 +216,9 @@
       <plugin>gazebo_ros2_control/GazeboSystem</plugin>
     </hardware>
-    <joint name="head_swivel">
-      <command_interface name="position" />
-      <command_interface name="velocity" />
-      <state_interface name="position"/>
-      <state_interface name="velocity"/>
-    </joint>
+    <joint name="head_swivel" />
   </ros2_control>
   <gazebo>
     <plugin filename="libgazebo_ros2_control.so" name="gazebo_ros2_control">
-      <parameters>$(find urdf_sim_tutorial)/config/head.yaml</parameters>
+      <parameters>$(find urdf_sim_tutorial)/config/09a-minimal.yaml</parameters>
     </plugin>
   </gazebo>

File: urdf/10-firsttransmission.urdf.xacro (robot description, xacro)
@@ -7,5 +7,4 @@
   <xacro:property name="baselen" value="0.4" />
   <xacro:property name="wheeldiam" value="0.07" />
-  <xacro:property name="pi" value="3.1415" />
   <material name="blue">
     <color rgba="0 0 0.8 1"/>
@@ -20,5 +19,5 @@
     <inertial>
       <mass value="${mass}" />
-      <inertia ixx="1.0" ixy="0.0" ixz="0.0" iyy="1.0" iyz="0.0" izz="1.0" />
+      <inertia ixx="1e-3" ixy="0.0" ixz="0.0" iyy="1e-3" iyz="0.0" izz="1e-3" />
     </inertial>
   </xacro:macro>
@@ -193,15 +192,4 @@
     <origin xyz="0 0 ${bodylen/2}"/>
   </joint>
-  <!-- This block connects the head_swivel joint to an actuator (motor), which informs both
-  simulation and visualization of the robot -->
-  <transmission name="head_swivel_trans">
-    <type>transmission_interface/SimpleTransmission</type>
-    <actuator name="$head_swivel_motor">
-      <mechanicalReduction>1</mechanicalReduction>
-    </actuator>
-    <joint name="head_swivel">
-      <hardwareInterface>PositionJointInterface</hardwareInterface>
-    </joint>
-  </transmission>
   <link name="box">
     <visual>
@@ -224,8 +212,18 @@
     <origin xyz="${.707*width+0.04} 0 ${.707*width}"/>
   </joint>
-  <!-- Gazebo plugin for ROS Control -->
+  <ros2_control name="GazeboSystem" type="system">
+    <hardware>
+      <plugin>gazebo_ros2_control/GazeboSystem</plugin>
+    </hardware>
+    <joint name="head_swivel">
+      <command_interface name="position" />
+      <command_interface name="velocity" />
+      <state_interface name="position"/>
+      <state_interface name="velocity"/>
+    </joint>
+  </ros2_control>
   <gazebo>
-    <plugin name="gazebo_ros_control" filename="libgazebo_ros_control.so">
-      <robotNamespace>/</robotNamespace>
+    <plugin filename="libgazebo_ros2_control.so" name="gazebo_ros2_control">
+      <parameters>$(find urdf_sim_tutorial)/config/head.yaml</parameters>
     </plugin>
   </gazebo>

File: urdf/12a-mimic-gripper.urdf.xacro (robot description, xacro)
@@ -1,4 +1,4 @@
 <?xml version="1.0"?>
-<robot name="first_transmission_with_limits" xmlns:xacro="http://ros.org/wiki/xacro">
+<robot name="gripper_controller" xmlns:xacro="http://ros.org/wiki/xacro">
   <xacro:property name="width" value="0.2" />
   <xacro:property name="leglen" value="0.6" />
@@ -111,4 +111,6 @@
     <limit effort="1000.0" lower="-${width*2-.02}" upper="0" velocity="0.5"/>
     <origin rpy="0 0 0" xyz="${width-.01} 0 0.2"/>
+    <limit effort="30" velocity="0.2"/>
+    <dynamics damping="0.0" friction="0.0"/>
   </joint>
   <link name="gripper_pole">
@@ -127,6 +129,7 @@
     <xacro:default_inertial mass="0.05"/>
   </link>
-  <xacro:macro name="gripper" params="prefix reflect">
+  <xacro:macro name="gripper" params="prefix reflect *extra_tag">
     <joint name="${prefix}_gripper_joint" type="revolute">
+      <xacro:insert_block name="extra_tag" />
       <axis xyz="0 0 ${reflect}"/>
       <limit effort="1000.0" lower="0.0" upper="0.548" velocity="0.5"/>
@@ -134,4 +137,6 @@
       <parent link="gripper_pole"/>
       <child link="${prefix}_gripper"/>
+      <limit effort="30" velocity="1.0"/>
+      <dynamics damping="0.0" friction="0.0"/>
     </joint>
     <link name="${prefix}_gripper">
@@ -170,6 +175,10 @@
     </link>
   </xacro:macro>
-  <xacro:gripper prefix="left" reflect="1" />
-  <xacro:gripper prefix="right" reflect="-1" />
+  <xacro:gripper prefix="left" reflect="1">
+    <dynamics damping="0.0" friction="0.0"/>
+  </xacro:gripper>
+  <xacro:gripper prefix="right" reflect="-1">
+     <mimic joint="left_gripper_joint"/>
+  </xacro:gripper>
   <link name="head">
     <visual>
@@ -192,4 +201,5 @@
     <origin xyz="0 0 ${bodylen/2}"/>
     <limit effort="30" velocity="1.0"/>
+    <dynamics damping="0.0" friction="0.0"/>
   </joint>
   <link name="box">
@@ -223,8 +233,28 @@
       <state_interface name="velocity"/>
     </joint>
+    <joint name="gripper_extension">
+      <command_interface name="position" />
+      <command_interface name="velocity" />
+      <state_interface name="position"/>
+      <state_interface name="velocity"/>
+    </joint>
+    <joint name="left_gripper_joint">
+      <command_interface name="position" />
+      <command_interface name="velocity" />
+      <state_interface name="position"/>
+      <state_interface name="velocity"/>
+    </joint>
+    <joint name="right_gripper_joint">
+      <command_interface name="position" />
+      <command_interface name="velocity" />
+      <state_interface name="position"/>
+      <state_interface name="velocity"/>
+      <param name="mimic">left_gripper_joint</param>
+      <param name="multiplier">1</param>
+    </joint>
   </ros2_control>
   <gazebo>
     <plugin filename="libgazebo_ros2_control.so" name="gazebo_ros2_control">
-      <parameters>$(find urdf_sim_tutorial)/config/head.yaml</parameters>
+      <parameters>$(find urdf_sim_tutorial)/config/mimic-gripper.yaml</parameters>
     </plugin>
   </gazebo>

File: urdf/13-diffdrive.urdf.xacro (robot description, xacro)
@@ -1,4 +1,4 @@
 <?xml version="1.0"?>
-<robot name="roscontrol" xmlns:xacro="http://ros.org/wiki/xacro">
+<robot name="diff_drive" xmlns:xacro="http://ros.org/wiki/xacro">
   <xacro:property name="width" value="0.2" />
   <xacro:property name="leglen" value="0.6" />
@@ -7,5 +7,4 @@
   <xacro:property name="baselen" value="0.4" />
   <xacro:property name="wheeldiam" value="0.07" />
-  <xacro:property name="pi" value="3.1415" />
   <material name="blue">
     <color rgba="0 0 0.8 1"/>
@@ -20,5 +19,5 @@
     <inertial>
       <mass value="${mass}" />
-      <inertia ixx="1.0" ixy="0.0" ixz="0.0" iyy="1.0" iyz="0.0" izz="1.0" />
+      <inertia ixx="1e-3" ixy="0.0" ixz="0.0" iyy="1e-3" iyz="0.0" izz="1e-3" />
     </inertial>
   </xacro:macro>
@@ -60,24 +59,4 @@
       <origin xyz="${baselen*reflect/3} 0 -${wheeldiam/2+.05}" rpy="0 0 0"/>
     </joint>
-    <!-- This block provides the simulator (Gazebo) with information on a few additional
-    physical properties. See http://gazebosim.org/tutorials/?tut=ros_urdf for more-->
-    <gazebo reference="${prefix}_${suffix}_wheel">
-      <mu1 value="200.0"/>
-      <mu2 value="100.0"/>
-      <kp value="10000000.0" />
-      <kd value="1.0" />
-      <material>Gazebo/Grey</material>
-    </gazebo>
-    <!-- This block connects the wheel joint to an actuator (motor), which informs both
-    simulation and visualization of the robot -->
-    <transmission name="${prefix}_${suffix}_wheel_trans">
-      <type>transmission_interface/SimpleTransmission</type>
-      <actuator name="${prefix}_${suffix}_wheel_motor">
-        <mechanicalReduction>1</mechanicalReduction>
-      </actuator>
-      <joint name="${prefix}_${suffix}_wheel_joint">
-        <hardwareInterface>VelocityJointInterface</hardwareInterface>
-      </joint>
-    </transmission>
   </xacro:macro>
   <xacro:macro name="leg" params="prefix reflect">
@@ -150,15 +129,7 @@
     <xacro:default_inertial mass="0.05"/>
   </link>
-  <transmission name="gripper_extension_trans">
-    <type>transmission_interface/SimpleTransmission</type>
-    <actuator name="gripper_extension_motor">
-      <mechanicalReduction>1</mechanicalReduction>
-    </actuator>
-    <joint name="gripper_extension">
-      <hardwareInterface>PositionJointInterface</hardwareInterface>
-    </joint>
-  </transmission>
-  <xacro:macro name="gripper" params="prefix reflect">
+  <xacro:macro name="gripper" params="prefix reflect *extra_tag">
     <joint name="${prefix}_gripper_joint" type="revolute">
+      <xacro:insert_block name="extra_tag" />
       <axis xyz="0 0 ${reflect}"/>
       <limit effort="1000.0" lower="0.0" upper="0.548" velocity="0.5"/>
@@ -184,13 +155,4 @@
       <xacro:default_inertial mass="0.05"/>
     </link>
-    <transmission name="${prefix}_gripper_trans">
-      <type>transmission_interface/SimpleTransmission</type>
-      <actuator name="${prefix}_gripper_motor">
-        <mechanicalReduction>1</mechanicalReduction>
-      </actuator>
-      <joint name="${prefix}_gripper_joint">
-        <hardwareInterface>PositionJointInterface</hardwareInterface>
-      </joint>
-    </transmission>
     <joint name="${prefix}_tip_joint" type="fixed">
       <parent link="${prefix}_gripper"/>
@@ -213,6 +175,10 @@
     </link>
   </xacro:macro>
-  <xacro:gripper prefix="left" reflect="1" />
-  <xacro:gripper prefix="right" reflect="-1" />
+  <xacro:gripper prefix="left" reflect="1">
+    <dynamics damping="0.0" friction="0.0"/>
+  </xacro:gripper>
+  <xacro:gripper prefix="right" reflect="-1">
+     <mimic joint="left_gripper_joint"/>
+  </xacro:gripper>
   <link name="head">
     <visual>
@@ -237,15 +203,4 @@
     <dynamics damping="0.0" friction="0.0"/>
   </joint>
-  <!-- This block connects the head_swivel joint to an actuator (motor), which informs both
-  simulation and visualization of the robot -->
-  <transmission name="head_swivel_trans">
-    <type>transmission_interface/SimpleTransmission</type>
-    <actuator name="$head_swivel_motor">
-      <mechanicalReduction>1</mechanicalReduction>
-    </actuator>
-    <joint name="head_swivel">
-      <hardwareInterface>PositionJointInterface</hardwareInterface>
-    </joint>
-  </transmission>
   <link name="box">
     <visual>
@@ -268,8 +223,58 @@
     <origin xyz="${.707*width+0.04} 0 ${.707*width}"/>
   </joint>
-  <!-- Gazebo plugin for ROS Control -->
+  <ros2_control name="GazeboSystem" type="system">
+    <hardware>
+      <plugin>gazebo_ros2_control/GazeboSystem</plugin>
+    </hardware>
+    <joint name="head_swivel">
+      <command_interface name="position" />
+      <command_interface name="velocity" />
+      <state_interface name="position"/>
+      <state_interface name="velocity"/>
+    </joint>
+    <joint name="gripper_extension">
+      <command_interface name="position" />
+      <command_interface name="velocity" />
+      <state_interface name="position"/>
+      <state_interface name="velocity"/>
+    </joint>
+    <joint name="left_gripper_joint">
+      <command_interface name="position" />
+      <command_interface name="velocity" />
+      <state_interface name="position"/>
+      <state_interface name="velocity"/>
+    </joint>
+    <joint name="right_gripper_joint">
+      <command_interface name="position" />
+      <command_interface name="velocity" />
+      <state_interface name="position"/>
+      <state_interface name="velocity"/>
+      <param name="mimic">left_gripper_joint</param>
+      <param name="multiplier">1</param>
+    </joint>
+    <joint name="left_front_wheel_joint">
+      <command_interface name="velocity" />
+      <state_interface name="position"/>
+      <state_interface name="velocity"/>
+    </joint>
+    <joint name="left_back_wheel_joint">
+      <command_interface name="velocity" />
+      <state_interface name="position"/>
+      <state_interface name="velocity"/>
+    </joint>
+    <joint name="right_front_wheel_joint">
+      <command_interface name="velocity" />
+      <state_interface name="position"/>
+      <state_interface name="velocity"/>
+    </joint>
+    <joint name="right_back_wheel_joint">
+      <command_interface name="velocity" />
+      <state_interface name="position"/>
+      <state_interface name="velocity"/>
+    </joint>
+  </ros2_control>
   <gazebo>
-    <plugin name="gazebo_ros_control" filename="libgazebo_ros_control.so">
-      <robotNamespace>/</robotNamespace>
+    <plugin filename="libgazebo_ros2_control.so" name="gazebo_ros2_control">
+      <parameters>$(find urdf_sim_tutorial)/config/diffdrive.yaml</parameters>
     </plugin>
   </gazebo>
